Commit message: New stable version of USV plugin and support packages

File: urdf/kingfisher_urdf.xacro (robot description, xacro)
@@ -29,117 +29,80 @@
 This program contains the description of the robot base model for the Clearpath Kingfisher
 -->
-<robot
-    xmlns:xi="http://www.w3.org/2001/XInclude"
-    xmlns:gazebo="http://playerstage.sourceforge.net/gazebo/xmlschema/#gz"
-    xmlns:model="http://playerstage.sourceforge.net/gazebo/xmlschema/#model"
-    xmlns:sensor="http://playerstage.sourceforge.net/gazebo/xmlschema/#sensor"
-    xmlns:body="http://playerstage.sourceforge.net/gazebo/xmlschema/#body"
-    xmlns:geom="http://playerstage.sourceforge.net/gazebo/xmlschema/#geom"
-    xmlns:joint="http://playerstage.sourceforge.net/gazebo/xmlschema/#joint"
-    xmlns:controller="http://playerstage.sourceforge.net/gazebo/xmlschema/#controller"
-    xmlns:interface="http://playerstage.sourceforge.net/gazebo/xmlschema/#interface"
-    xmlns:rendering="http://playerstage.sourceforge.net/gazebo/xmlschema/#rendering"
-    xmlns:renderable="http://playerstage.sourceforge.net/gazebo/xmlschema/#renderable"
-    xmlns:physics="http://playerstage.sourceforge.net/gazebo/xmlschema/#physics"
-    xmlns:xacro="http://ros.org/wiki/xacro" name="kingfisher">
-    <!-- Included URDF/XACRO Files -->
-    <xacro:include filename="$(find kingfisher_description)/urdf/materials.urdf.xacro" />
-    <!-- Replace original Kingfisher file with new one with minimial inertia-->
-    <xacro:include filename="$(find kingfisher_gazebo)/urdf/parts.mininertia.urdf.xacro" />
-    <!-- PROPERTY LIST -->
-    <!--All units in m-kg-s-radians unit system -->
-    <property name="M_PI" value="3.1415926535897931" />
-    <!-- BASE-FOOTPRINT -->
-    <!-- base_fotporint is a fictitious link(frame) that is on the ground right below base_link origin, navigation stack depends on this frame -->
-    <link name="base_footprint">
-        <inertial>
-            <mass value="0.0001" />
-            <origin xyz="0 0 0" />
-            <inertia ixx="0.0001" ixy="0.0" ixz="0.0"
-                iyy="0.0001" iyz="0.0"
-                izz="0.0001" />
-        </inertial>
-        <visual>
-            <origin xyz="0 0 0" rpy="0 0 0" />
-            <geometry>
-                <box size="0.001 0.001 0.001" />
-            </geometry>
-        </visual>
-    </link>
-    <gazebo reference="base_footprint">
-        <turnGravityOff>false</turnGravityOff>
-    </gazebo>
-    <joint name="base_footprint_joint" type="fixed">
+<robot name="kingfisher" xmlns:xacro="http://ros.org/wiki/xacro">
+  <!-- Included URDF/XACRO Files -->
+  <xacro:include filename="$(find kingfisher_description)/urdf/materials.urdf.xacro" />
+  <!-- Replace original Kingfisher file with new one with minimial inertia-->
+  <xacro:include filename="$(find kingfisher_gazebo)/urdf/parts.mininertia.urdf.xacro" />
+  <!-- PROPERTY LIST -->
+  <!--All units in m-kg-s-radians unit system -->
+  <property name="M_PI" value="3.1415926535897931" />
+  <!-- BASE-FOOTPRINT -->
+  <!-- base_fotporint is a fictitious link(frame) that is on the ground right below base_link origin, navigation stack depends on this frame -->
+  <link name="base_footprint">
+    <inertial>
+      <mass value="1e-5" />
+      <origin xyz="0 0 0" />
+      <inertia ixx="1e-6" ixy="0.0" ixz="0.0"
+	       iyy="1e-6" iyz="0.0"
+	       izz="1e-6" />
+    </inertial>
+    <visual>
+      <origin xyz="0 0 0" rpy="0 0 0" />
+      <geometry>
+	<box size="0.001 0.001 0.001" />
+      </geometry>
+    </visual>
+  </link>
+  <gazebo reference="base_footprint">
+    <turnGravityOff>false</turnGravityOff>
+  </gazebo>
+  <!-- BASE-LINK -->
+  <!--Actual body/chassis of the robot-->
+  <link name="base_link">
+    <inertial>
+      <mass value="29" />
+      <!--This is the pose of the inertial reference frame, relative to the link reference frame. The origin of the inertial reference frame needs to be at the center of gravity. The axes of the inertial reference frame do not need to be aligned with the principal axes of the inertia.-->
+      <origin xyz="0 0 0" />
+      <!--The 3x3 rotational inertia matrix. Because the rotational inertia matrix is symmetric, only 6 above-diagonal elements of this matrix are specified here, using the attributes ixx, ixy, ixz, iyy, iyz, izz.-->
+      <inertia ixx="10" ixy="0" ixz="0" iyy="10" iyz="0" izz="10" />
+    </inertial>
+    <visual>
+      <origin xyz="0 0 0" rpy="${M_PI/2} 0 ${M_PI/2}" />
+      <geometry>
+	<mesh filename="package://kingfisher_description/meshes/kingfisher_base.stl" />
+      </geometry>
+      <material name="DarkGray" />
+    </visual>
+    <collision>
+      <origin xyz="0 0 0" rpy="0 0 0" />
+      <geometry>
+	<box size = "0.1 0.1 0.1"/> <!--making it slightly bigger in x and z direction-->
+      </geometry>
+    </collision>
+  </link>
+  <joint name="base_footprint_joint" type="fixed">
     <origin xyz="0 0 0" rpy="0 0 0" />
-        <parent link="base_footprint"/>
-        <child link="base_link" />
-    </joint>
-    <!-- BASE-LINK -->
-    <!--Actual body/chassis of the robot-->
-    <link name="base_link">
-        <inertial>
-            <mass value="29" />
-            <!--This is the pose of the inertial reference frame, relative to the link reference frame. The origin of the inertial reference frame needs to be at the center of gravity. The axes of the inertial reference frame do not need to be aligned with the principal axes of the inertia.-->
-            <origin xyz="0 0 0" />
-            <!--The 3x3 rotational inertia matrix. Because the rotational inertia matrix is symmetric, only 6 above-diagonal elements of this matrix are specified here, using the attributes ixx, ixy, ixz, iyy, iyz, izz.-->
-            <inertia ixx="10" ixy="0" ixz="0" iyy="10" iyz="0" izz="10" />
-        </inertial>
-        <visual>
-            <origin xyz="0 0 0" rpy="${M_PI/2} 0 ${M_PI/2}" />
-            <geometry>
-                <mesh filename="package://kingfisher_description/meshes/kingfisher_base.stl" />
-            </geometry>
-            <material name="DarkGray" />
-        </visual>
-        <collision>
-          <origin xyz="0 0 0" rpy="0 0 0" />
-          <geometry>
-                <box size = "0.1 0.1 0.1"/> <!--making it slightly bigger in x and z direction-->
-            </geometry>
-        </collision>
-    </link>
-    <gazebo reference="base_link">
-        <material>Gazebo/FlatBlack</material>
-        <turnGravityOff>false</turnGravityOff>
-    </gazebo>
-    <!-- Thruster Link, provides a place to apply thrust force-->
-    <link name="thrust_link">
-      <inertial>
-	<mass value="0.0001" />
-	<origin xyz="0 0 0" />
-	<inertia ixx="0.0001" ixy="0.0" ixz="0.0"
-		 iyy="0.0001" iyz="0.0"
-		 izz="0.0001" />
-      </inertial>
-      <visual>
-	<origin xyz="0 0 0" rpy="0 0 0" />
-	<geometry>
-	  <box size="0.001 0.001 0.001" />
-	</geometry>
-      </visual>
-    </link>
-   <gazebo reference="thrust_link">
-     <turnGravityOff>false</turnGravityOff>
-   </gazebo>
-    <joint name="thrust_joint" type="fixed">
-    <origin xyz="0 0 -0.5" rpy="0 0 0" />
-        <parent link="base_link"/>
-        <child link="thrust_link" />
-    </joint>
-    <!-- PANEL-LINKS -->
-    <!-- Top Plate -->
-    <kingfisher_part parent="base_footprint" name="left_panel" mesh="left_panel"
-          translateX="0.0" translateY="-0.35" translateZ="0.05"
-          rotateX="${M_PI/2}" rotateY="0.0" rotateZ="${M_PI/2}"
-          color="Yellow" />
-    <gazebo reference="base_footprint_left_panel_part">
-        <material>Gazebo/Yellow</material>
-    </gazebo>
-    <kingfisher_part parent="base_footprint" name="right_panel" mesh="right_panel"
-          translateX="0.0" translateY="0.35" translateZ="0.05"
-          rotateX="${M_PI/2}" rotateY="0.0" rotateZ="${-M_PI/2}"
-          color="Yellow" />
-    <gazebo reference="base_footprint_right_panel_part">
-        <material>Gazebo/Yellow</material>
-    </gazebo>
+    <parent link="base_footprint"/>
+    <child link="base_link" />
+  </joint>
+  <gazebo reference="base_link">
+    <material>Gazebo/FlatBlack</material>
+    <turnGravityOff>false</turnGravityOff>
+  </gazebo>
+  <!-- PANEL-LINKS -->
+  <!-- Top Plate -->
+  <kingfisher_part parent="base_footprint" name="left_panel" mesh="left_panel"
+		   translateX="0.0" translateY="-0.35" translateZ="0.05"
+		   rotateX="${M_PI/2}" rotateY="0.0" rotateZ="${M_PI/2}"
+		   color="Yellow" />
+  <gazebo reference="base_footprint_left_panel_part">
+    <material>Gazebo/Yellow</material>
+  </gazebo>
+  <kingfisher_part parent="base_footprint" name="right_panel" mesh="right_panel"
+		   translateX="0.0" translateY="0.35" translateZ="0.05"
+		   rotateX="${M_PI/2}" rotateY="0.0" rotateZ="${-M_PI/2}"
+		   color="Yellow" />
+  <gazebo reference="base_footprint_right_panel_part">
+    <material>Gazebo/Yellow</material>
+  </gazebo>
 </robot>

Commit message: Working lake world - tweak of USV plugin and xacro collision description

File: urdf/kingfisher_urdf.xacro (robot description, xacro)
@@ -77,5 +77,5 @@
       <origin xyz="0 0 0" rpy="0 0 0" />
       <geometry>
-	<box size = "0.1 0.1 0.1"/> <!--making it slightly bigger in x and z direction-->
+	<box size = "1.35 0.98 0.2"/> <!--making it slightly bigger in x and z direction-->
       </geometry>
     </collision>

Commit message: change origin of kingfisher visual to correspond with water line

File: urdf/kingfisher_urdf.xacro (robot description, xacro)
@@ -37,4 +37,5 @@
   <!--All units in m-kg-s-radians unit system -->
   <property name="M_PI" value="3.1415926535897931" />
+  <property name="HH" value="0.09" />
   <!-- BASE-FOOTPRINT -->
   <!-- base_fotporint is a fictitious link(frame) that is on the ground right below base_link origin, navigation stack depends on this frame -->
@@ -42,5 +43,5 @@
     <inertial>
       <mass value="1e-5" />
-      <origin xyz="0 0 0" />
+      <origin xyz="0 0 ${HH} " />
       <inertia ixx="1e-6" ixy="0.0" ixz="0.0"
 	       iyy="1e-6" iyz="0.0"
@@ -48,5 +49,5 @@
     </inertial>
     <visual>
-      <origin xyz="0 0 0" rpy="0 0 0" />
+      <origin xyz="0 0 ${HH}" rpy="0 0 0" />
       <geometry>
 	<box size="0.001 0.001 0.001" />
@@ -63,10 +64,10 @@
       <mass value="29" />
       <!--This is the pose of the inertial reference frame, relative to the link reference frame. The origin of the inertial reference frame needs to be at the center of gravity. The axes of the inertial reference frame do not need to be aligned with the principal axes of the inertia.-->
-      <origin xyz="0 0 0" />
+      <origin xyz="0 0 ${HH}" />
       <!--The 3x3 rotational inertia matrix. Because the rotational inertia matrix is symmetric, only 6 above-diagonal elements of this matrix are specified here, using the attributes ixx, ixy, ixz, iyy, iyz, izz.-->
       <inertia ixx="10" ixy="0" ixz="0" iyy="10" iyz="0" izz="10" />
     </inertial>
     <visual>
-      <origin xyz="0 0 0" rpy="${M_PI/2} 0 ${M_PI/2}" />
+      <origin xyz="0 0 ${HH}" rpy="${M_PI/2} 0 ${M_PI/2}" />
       <geometry>
 	<mesh filename="package://kingfisher_description/meshes/kingfisher_base.stl" />
@@ -82,5 +83,5 @@
   </link>
   <joint name="base_footprint_joint" type="fixed">
-    <origin xyz="0 0 0" rpy="0 0 0" />
+    <origin xyz="0 0 ${HH}" rpy="0 0 0" />
     <parent link="base_footprint"/>
     <child link="base_link" />
@@ -93,5 +94,5 @@
   <!-- Top Plate -->
   <kingfisher_part parent="base_footprint" name="left_panel" mesh="left_panel"
-		   translateX="0.0" translateY="-0.35" translateZ="0.05"
+		   translateX="0.0" translateY="-0.35" translateZ="${0.05+HH*2}"
 		   rotateX="${M_PI/2}" rotateY="0.0" rotateZ="${M_PI/2}"
 		   color="Yellow" />
@@ -100,5 +101,5 @@
   </gazebo>
   <kingfisher_part parent="base_footprint" name="right_panel" mesh="right_panel"
-		   translateX="0.0" translateY="0.35" translateZ="0.05"
+		   translateX="0.0" translateY="0.35" translateZ="${0.05+HH*2}"
 		   rotateX="${M_PI/2}" rotateY="0.0" rotateZ="${-M_PI/2}"
 		   color="Yellow" />
