Commit message: changing xacro syntax for kinetic

File: urdf/base.urdf.xacro (robot description, xacro)
@@ -44,5 +44,5 @@
     <!-- PROPERTY LIST -->
     <!--All units in m-kg-s-radians unit system -->
-    <property name="M_PI" value="3.1415926535897931" />
+    <xacro:property name="M_PI" value="3.1415926535897931" />
     <!-- BASE-FOOTPRINT -->
     <!-- base_footprint is a fictitious link(frame) that is on the ground right below base_link origin, navigation stack depends on this frame -->

File: urdf/base2.urdf.xacro (robot description, xacro)
@@ -44,5 +44,5 @@
     <!-- PROPERTY LIST -->
     <!--All units in m-kg-s-radians unit system -->
-    <property name="M_PI" value="3.1415926535897931" />
+    <xacro:property name="M_PI" value="3.1415926535897931" />
     <xacro:macro name="kingfisher_base">
     <!-- BASE-FOOTPRINT -->

File: urdf/base_urdf.xacro (robot description, xacro)
@@ -44,5 +44,5 @@
     <!-- PROPERTY LIST -->
     <!--All units in m-kg-s-radians unit system -->
-    <property name="M_PI" value="3.1415926535897931" />
+    <xacro:property name="M_PI" value="3.1415926535897931" />
     <xacro:macro name="kingfisher_base">
     <!-- BASE-FOOTPRINT -->

File: urdf/kingfisher_urdf.xacro (robot description, xacro)
@@ -30,4 +30,5 @@
 -->
 <robot name="kingfisher" xmlns:xacro="http://ros.org/wiki/xacro">
+  <xacro:macro name="kingfisher_base">
   <!-- Included URDF/XACRO Files -->
   <xacro:include filename="$(find kingfisher_description)/urdf/materials.urdf.xacro" />
@@ -36,6 +37,6 @@
   <!-- PROPERTY LIST -->
   <!--All units in m-kg-s-radians unit system -->
-  <property name="M_PI" value="3.1415926535897931" />
-  <property name="HH" value="0.09" />
+  <xacro:property name="M_PI" value="3.1415926535897931" />
+  <xacro:property name="HH" value="0.09" />
   <!-- BASE-FOOTPRINT -->
   <!-- base_fotporint is a fictitious link(frame) that is on the ground right below base_link origin, navigation stack depends on this frame -->
@@ -139,3 +140,4 @@
     <turnGravityOff>false</turnGravityOff>
   </gazebo>
+</xacro:macro>
 </robot>

File: urdf/kingfisher_urdf_base.xacro (robot description, xacro)
@@ -36,6 +36,6 @@
   <!-- PROPERTY LIST -->
   <!--All units in m-kg-s-radians unit system -->
-  <property name="M_PI" value="3.1415926535897931" />
-  <property name="HH" value="0.09" />
+  <xacro:property name="M_PI" value="3.1415926535897931" />
+  <xacro:property name="HH" value="0.09" />
   <!-- BASE-FOOTPRINT -->
   <!-- base_fotporint is a fictitious link(frame) that is on the ground right below base_link origin, navigation stack depends on this frame -->

File: urdf/kingfisher_urdf_camera.xacro (robot description, xacro)
@@ -36,6 +36,6 @@
   <!-- PROPERTY LIST -->
   <!--All units in m-kg-s-radians unit system -->
-  <property name="M_PI" value="3.1415926535897931" />
-  <property name="HH" value="0.09" />
+  <xacro:property name="M_PI" value="3.1415926535897931" />
+  <xacro:property name="HH" value="0.09" />
   <!-- BASE-FOOTPRINT -->
   <!-- base_fotporint is a fictitious link(frame) that is on the ground right below base_link origin, navigation stack depends on this frame -->

File: urdf/parts.mininertia.urdf.xacro (robot description, xacro)
@@ -36,18 +36,18 @@
 	xmlns:interface="http://playerstage.sourceforge.net/gazebo/xmlschema/#interface"
 	xmlns:xacro="http://ros.org/wiki/xacro" name="kingfisher_part">
-	<property name="x_com" value="0.00000000" /> <!-- com : center of mass -->
-	<property name="y_com" value="0.00000000" /> <!-- com : center of mass -->
-	<property name="z_com" value="0.00000000" /> <!-- com : center of mass -->
-	<property name="x_size" value="1.0" />
-	<property name="y_size" value="1.0" />
-	<property name="z_size" value="1.0" />
-	<property name="min_inertia" value="0.00001"/>
-	<property name="mass" value="${min_inertia}" /> <!-- in kg-->
-	<property name="ixx_com_cs" value="${min_inertia}" /> <!-- at center of mass aligned with coordinate system, kg*m^2-->
-	<property name="ixy_com_cs" value="0.0" /> <!-- at center of mass aligned with coordinate system, kg*m^2-->
-	<property name="ixz_com_cs" value="0.0" /> <!-- at center of mass aligned with coordinate system, kg*m^2-->
-	<property name="iyy_com_cs" value="${min_inertia}" /> <!-- at center of mass aligned with coordinate system, kg*m^2-->
-	<property name="iyz_com_cs" value="0.00" /> <!-- at center of mass aligned with coordinate system, kg*m^2-->
-	<property name="izz_com_cs" value="${min_inertia}" /> <!-- at center of mass aligned with coordinate system, kg*m^2-->
+	<xacro:property name="x_com" value="0.00000000" /> <!-- com : center of mass -->
+	<xacro:property name="y_com" value="0.00000000" /> <!-- com : center of mass -->
+	<xacro:property name="z_com" value="0.00000000" /> <!-- com : center of mass -->
+	<xacro:property name="x_size" value="1.0" />
+	<xacro:property name="y_size" value="1.0" />
+	<xacro:property name="z_size" value="1.0" />
+	<xacro:property name="min_inertia" value="0.00001"/>
+	<xacro:property name="mass" value="${min_inertia}" /> <!-- in kg-->
+	<xacro:property name="ixx_com_cs" value="${min_inertia}" /> <!-- at center of mass aligned with coordinate system, kg*m^2-->
+	<xacro:property name="ixy_com_cs" value="0.0" /> <!-- at center of mass aligned with coordinate system, kg*m^2-->
+	<xacro:property name="ixz_com_cs" value="0.0" /> <!-- at center of mass aligned with coordinate system, kg*m^2-->
+	<xacro:property name="iyy_com_cs" value="${min_inertia}" /> <!-- at center of mass aligned with coordinate system, kg*m^2-->
+	<xacro:property name="iyz_com_cs" value="0.00" /> <!-- at center of mass aligned with coordinate system, kg*m^2-->
+	<xacro:property name="izz_com_cs" value="${min_inertia}" /> <!-- at center of mass aligned with coordinate system, kg*m^2-->
 	<xacro:macro name="kingfisher_part" params="parent name mesh translateX translateY translateZ rotateX rotateY rotateZ color">
 		<joint name="${parent}_${name}_joint" type="fixed">
