Commit message: functional version with IMU and GPS simulation

File: urdf/base_gazebo.xacro (robot description, xacro)
@@ -6,4 +6,8 @@
   <!-- Defines the "usv_gazebo" macro which implements the plugin for USV dynamics -->
   <xacro:include filename="$(find kingfisher_gazebo)/urdf/usv_gazebo.xacro" />
+  <!-- Defines the macro for simulated GPS -->
+  <xacro:include filename="$(find kingfisher_gazebo)/urdf/gps_gazebo.xacro" />
+  <!-- Defines the macro for simulated IMU -->
+  <xacro:include filename="$(find kingfisher_gazebo)/urdf/imu_gazebo.xacro" />
   <!-- Call the macros defined above -->
   <!-- includes basic description witout plugins -->
@@ -11,3 +15,10 @@
   <!-- USV dynamic model -->
   <xacro:usv_gazebo name="kingfisher"/>
+  <!-- Optional sensor plugins -->
+  <xacro:if value="$(arg gps)">
+    <xacro:kingfisher_gps_gazebo name="kingfisher"/>
+  </xacro:if>
+  <xacro:if value="$(arg imu)">
+    <xacro:kingfisher_imu_gazebo name="kingfisher"/>
+  </xacro:if>
 </robot>

File: urdf/base_urdf.xacro (robot description, xacro)
@@ -115,5 +115,4 @@
         <material>Gazebo/Yellow</material>
     </gazebo>
-    <!--Gazebo Plugin for simulating Kingfisher dynamics-->
     </xacro:macro>
 </robot>

File: urdf/gps_gazebo.xacro (robot description, xacro)
@@ -1,5 +1,5 @@
 <?xml version="1.0"?>
 <robot xmlns:xacro="http://ros.org/wiki/xacro">
-  <xacro:macro name="gps_gazebo" params="name">
+  <xacro:macro name="kingfisher_gps_gazebo" params="name">
     <gazebo>
       <plugin name="gps_plugin_${name}" filename="libhector_gazebo_ros_gps.so">

File: urdf/imu_gazebo.xacro (robot description, xacro)
@@ -1,5 +1,5 @@
 <?xml version="1.0"?>
 <robot xmlns:xacro="http://ros.org/wiki/xacro">
-  <xacro:macro name="imu_gazebo" params="name">
+  <xacro:macro name="kingfisher_imu_gazebo" params="name">
     <gazebo>
       <!-- Either plugin should work -->
@@ -13,5 +13,5 @@
 	<serviceName>imu_service</serviceName>
 	<gaussianNoise>0.0</gaussianNoise>
-	<updateRate>20.0</updateRate>
+	<updateRate>10.0</updateRate>
       </plugin>
     </gazebo>

Commit message: preparation for messing with URDF definition

File: urdf/base_gazebo.xacro (robot description, xacro)
@@ -6,4 +6,6 @@
   <!-- Defines the "usv_gazebo" macro which implements the plugin for USV dynamics -->
   <xacro:include filename="$(find usv_gazebo_plugins)/urdf/usv_gazebo_dynamics_plugin.xacro" />
+  <!-- Testing old plugin -->
+  <!--<xacro:include filename="$(find kingfisher_plugins)/urdf/kingfisher_plugin.xacro" />-->
   <!-- Defines the macro for simulated GPS -->
   <xacro:include filename="$(find kingfisher_gazebo)/urdf/gps_gazebo.xacro" />

File: urdf/kingfisher_urdf.xacro (robot description, xacro)
@@ -51,5 +51,5 @@
     <property name="M_PI" value="3.1415926535897931" />
     <!-- BASE-FOOTPRINT -->
-    <!-- base_footprint is a fictitious link(frame) that is on the ground right below base_link origin, navigation stack depends on this frame -->
+    <!-- base_fotporint is a fictitious link(frame) that is on the ground right below base_link origin, navigation stack depends on this frame -->
     <link name="base_footprint">
         <inertial>
@@ -103,4 +103,28 @@
         <turnGravityOff>false</turnGravityOff>
     </gazebo>
+    <!-- Thruster Link, provides a place to apply thrust force-->
+    <link name="thrust_link">
+      <inertial>
+	<mass value="0.0001" />
+	<origin xyz="0 0 0" />
+	<inertia ixx="0.0001" ixy="0.0" ixz="0.0"
+		 iyy="0.0001" iyz="0.0"
+		 izz="0.0001" />
+      </inertial>
+      <visual>
+	<origin xyz="0 0 0" rpy="0 0 0" />
+	<geometry>
+	  <box size="0.001 0.001 0.001" />
+	</geometry>
+      </visual>
+    </link>
+   <gazebo reference="thrust_link">
+     <turnGravityOff>false</turnGravityOff>
+   </gazebo>
+    <joint name="thrust_joint" type="fixed">
+    <origin xyz="0 0 -0.5" rpy="0 0 0" />
+        <parent link="base_link"/>
+        <child link="thrust_link" />
+    </joint>
     <!-- PANEL-LINKS -->
     <!-- Top Plate -->

Commit message: toward del monte lake

File: urdf/base_gazebo.xacro (robot description, xacro)
@@ -3,10 +3,12 @@
        name="kingfisher">
   <!-- Defines the "kingfisher_base" macro -->
-  <!--<xacro:include filename="$(find kingfisher_gazebo)/urdf/kingfisher_urdf.xacro" />-->
-  <xacro:include filename="$(find kingfisher_gazebo)/urdf/kingfisher_urdf_camera.xacro" />-->
+  <xacro:include filename="$(find kingfisher_gazebo)/urdf/kingfisher_urdf.xacro" />
+  <!--<xacro:include filename="$(find kingfisher_gazebo)/urdf/kingfisher_urdf_camera.xacro" />-->
   <!-- Defines the "usv_gazebo" macro which implements the plugin for USV dynamics -->
   <xacro:include filename="$(find usv_gazebo_plugins)/urdf/usv_gazebo_dynamics_plugin.xacro" />
   <!-- Testing old plugin -->
   <!--<xacro:include filename="$(find kingfisher_plugins)/urdf/kingfisher_plugin.xacro" />-->
+  <!-- Defines the macro for including simulated camera -->
+  <xacro:include filename="$(find kingfisher_gazebo)/urdf/kingfisher_camera.xacro" />
   <!-- Defines the macro for simulated GPS -->
   <xacro:include filename="$(find kingfisher_gazebo)/urdf/gps_gazebo.xacro" />
@@ -30,3 +32,4 @@
     <xacro:kingfisher_p3d_gazebo name="kingfisher"/>
   </xacro:if>
+  <xacro:kingfisher_gazebo_camera name="kingfisher"/>
 </robot>

File: urdf/kingfisher_urdf.xacro (robot description, xacro)
@@ -76,5 +76,5 @@
     </visual>
     <collision>
-      <origin xyz="0 0 0" rpy="0 0 0" />
+      <origin xyz="0 0 ${HH}" rpy="0 0 0" />
       <geometry>
 	<box size = "1.35 0.98 0.2"/> <!--making it slightly bigger in x and z direction-->
@@ -107,3 +107,35 @@
     <material>Gazebo/Yellow</material>
   </gazebo>
+  <!-- Define a location for the camera to sit -->
+  <xacro:property name="camera_size" value="0.05" /> <!-- Size of square 'camera' box -->
+  <joint name="camera_joint" type="fixed">
+    <axis xyz="0 1 0" />
+    <origin xyz="0.32 0 0.2" rpy="0 0 0"/>
+    <parent link="base_link"/>
+    <child link="camera_link"/>
+  </joint>
+  <link name="camera_link">
+    <collision>
+      <origin xyz="0 0 0" rpy="0 0 0"/>
+      <geometry>
+	<box size="${camera_size} ${camera_size} ${camera_size}"/>
+      </geometry>
+    </collision>
+    <visual>
+      <origin xyz="0 0 0" rpy="0 0 0"/>
+      <geometry>
+	<box size="${camera_size} ${camera_size} ${camera_size}"/>
+      </geometry>
+      <material name="red"/>
+    </visual>
+    <inertial>
+      <mass value="1e-5" />
+      <origin xyz="0 0 0" rpy="0 0 0"/>
+      <inertia ixx="1e-6" ixy="0" ixz="0" iyy="1e-6" iyz="0" izz="1e-6" />
+    </inertial>
+  </link>
+  <gazebo reference="camera_link">
+    <material>Gazebo/Red</material>
+    <turnGravityOff>false</turnGravityOff>
+  </gazebo>
 </robot>

Commit message: changes to xacro to for indigo

File: urdf/base_gazebo.xacro (robot description, xacro)
@@ -2,4 +2,7 @@
 <robot xmlns:xacro="http://ros.org/wiki/xacro"
        name="kingfisher">
+  <xacro:property name="M_PI" value="3.1415926535897931" />
+  <xacro:property name="HH" value="0.09" />
+  <xacro:property name="camera_size" value="0.05" /> <!-- Size of square 'camera' box -->
   <!-- Defines the "kingfisher_base" macro -->
   <xacro:include filename="$(find kingfisher_gazebo)/urdf/kingfisher_urdf.xacro" />

File: urdf/kingfisher_urdf.xacro (robot description, xacro)
@@ -34,5 +34,7 @@
   <xacro:include filename="$(find kingfisher_description)/urdf/materials.urdf.xacro" />
   <!-- Replace original Kingfisher file with new one with minimial inertia-->
+  <!--
   <xacro:include filename="$(find kingfisher_gazebo)/urdf/parts.mininertia.urdf.xacro" />
+  -->
   <!-- PROPERTY LIST -->
   <!--All units in m-kg-s-radians unit system -->
@@ -44,5 +46,5 @@
     <inertial>
       <mass value="1e-5" />
-      <origin xyz="0 0 ${HH} " />
+      <origin xyz="0 0 0.09 " />
       <inertia ixx="1e-6" ixy="0.0" ixz="0.0"
 	       iyy="1e-6" iyz="0.0"
@@ -50,5 +52,5 @@
     </inertial>
     <visual>
-      <origin xyz="0 0 ${HH}" rpy="0 0 0" />
+      <origin xyz="0 0 0.09" rpy="0 0 0" />
       <geometry>
 	<box size="0.001 0.001 0.001" />
@@ -65,10 +67,10 @@
       <mass value="29" />
       <!--This is the pose of the inertial reference frame, relative to the link reference frame. The origin of the inertial reference frame needs to be at the center of gravity. The axes of the inertial reference frame do not need to be aligned with the principal axes of the inertia.-->
-      <origin xyz="0 0 ${HH}" />
+      <origin xyz="0 0 0.09" />
       <!--The 3x3 rotational inertia matrix. Because the rotational inertia matrix is symmetric, only 6 above-diagonal elements of this matrix are specified here, using the attributes ixx, ixy, ixz, iyy, iyz, izz.-->
       <inertia ixx="10" ixy="0" ixz="0" iyy="10" iyz="0" izz="10" />
     </inertial>
     <visual>
-      <origin xyz="0 0 ${HH}" rpy="${M_PI/2} 0 ${M_PI/2}" />
+      <origin xyz="0 0 0.09" rpy="${3.14159/2} 0 ${3.14159/2}" />
       <geometry>
 	<mesh filename="package://kingfisher_description/meshes/kingfisher_base.stl" />
@@ -77,5 +79,5 @@
     </visual>
     <collision>
-      <origin xyz="0 0 ${HH}" rpy="0 0 0" />
+      <origin xyz="0 0 0.09" rpy="0 0 0" />
       <geometry>
 	<box size = "1.35 0.98 0.2"/> <!--making it slightly bigger in x and z direction-->
@@ -84,5 +86,5 @@
   </link>
   <joint name="base_footprint_joint" type="fixed">
-    <origin xyz="0 0 ${HH}" rpy="0 0 0" />
+    <origin xyz="0 0 0.09" rpy="0 0 0" />
     <parent link="base_footprint"/>
     <child link="base_link" />
@@ -96,5 +98,5 @@
   <kingfisher_part parent="base_footprint" name="left_panel" mesh="left_panel"
 		   translateX="0.0" translateY="-0.35" translateZ="${0.05+HH*2}"
-		   rotateX="${M_PI/2}" rotateY="0.0" rotateZ="${M_PI/2}"
+		   rotateX="${3.14159/2}" rotateY="0.0" rotateZ="${3.14159/2}"
 		   color="Yellow" />
   <gazebo reference="base_footprint_left_panel_part">
@@ -103,5 +105,5 @@
   <kingfisher_part parent="base_footprint" name="right_panel" mesh="right_panel"
 		   translateX="0.0" translateY="0.35" translateZ="${0.05+HH*2}"
-		   rotateX="${M_PI/2}" rotateY="0.0" rotateZ="${-M_PI/2}"
+		   rotateX="${3.14159/2}" rotateY="0.0" rotateZ="${-3.14159/2}"
 		   color="Yellow" />
   <gazebo reference="base_footprint_right_panel_part">
